File: 12v_servo_driver.kicad_pcb (KiCad board)
At the start: 2 copper layers, 36.4 x 15 mm, 7 parts, among them J1 PWR/Signal, J2 Servo, U1 AMS1117-5.0

Commit message: Update gerber for RevB
Other:
- board text added: "Rev: B Servo Controller"
- board text removed: "Rev: A Servo Controller"
Changed lines of the file:
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@@
     (fp_line (start 5.95 6.25) (end 5.95 -1.35)
       (stroke (width 0.1) (type solid)) (layer "F.Fab"))
-    (pad "1" thru_hole roundrect (at 0 0 180) (size 1.2 1.75) (drill 0.75) (layers "*.Cu" "*.Mask") (roundrect_rratio 0.208333)
+    (pad "1" thru_hole roundrect (at 0 0 180) (size 1.2 1.75) (drill 0.75) (layers "*.Cu" "*.Mask") (roundrect_rratio 0.2083333333)
       (net 4 "/PWM") (pinfunction "Pin_1") (pintype "passive"))
     (pad "2" thru_hole oval (at 2 0 180) (size 1.2 1.75) (drill 0.75) (layers "*.Cu" "*.Mask")
@@
   (gr_arc (start 138.049 114.9985) (mid 134.1755 111.125) (end 138.049 107.2515)
     (stroke (width 0.05) (type solid)) (layer "Edge.Cuts"))
-  (gr_text "Rev: A Servo Controller" (at 151.9555 105.2068) (layer "B.SilkS")
+  (gr_text "Rev: B Servo Controller" (at 152.5 116.5) (layer "B.SilkS")
     (effects (font (size 1 1) (thickness 0.15)) (justify mirror))
   )
-  (gr_text "https://github.com/\ntheworkisthework/\n12v_servo_driver_module" (at 152.2603 108.5596) (layer "B.SilkS")
+  (gr_text "https://github.com/\ntheworkisthework/\n12v_servo_driver_module" (at 152.25 106.75) (layer "B.SilkS")
     (effects (font (size 1 1) (thickness 0.15)) (justify mirror))
   )
